File: pcb/mcu.kicad_sch (KiCad schematic)
At the start: 17 parts, among them J1 AVR-UPDI-6, U1 ATtiny1616-MNR

Commit message: Clean up and fixed attributes
Parts:
- removed TP10, TP11: ~, CRGM Mechanical:TestPoint_Pad_D1.0mm, symbol CRGM Connector:TestPoint
Connections:
- net PA6 renamed I2C_RESET
- net PA7 renamed I2C_INT
