File: pcb/module-base-attiny1616.kicad_sch (KiCad schematic)
At the start: 0 parts

Commit message: Clean up and fixed attributes
Connections:
- no-connect marks 0 -> 10
Other:
- sheet MCU ports: added I2C_INT, I2C_RESET; removed none
Changed lines of the file:
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@@
 		)
+	)
+	(no_connect
+		(at 162.56 45.72)
+	)
+	(no_connect
+		(at 162.56 38.1)
+	)
+	(no_connect
+		(at 147.32 53.34)
+	)
+	(no_connect
+		(at 152.4 53.34)
+	)
+	(no_connect
+		(at 162.56 40.64)
+	)
+	(no_connect
+		(at 149.86 53.34)
+	)
+	(no_connect
+		(at 162.56 27.94)
+	)
+	(no_connect
+		(at 162.56 48.26)
+	)
+	(no_connect
+		(at 162.56 35.56)
+	)
+	(no_connect
+		(at 162.56 43.18)
 	)
 	(wire
@@
 	(wire
 		(pts
+			(xy 111.76 38.1) (xy 127 38.1)
+		)
+		(stroke
+			(width 0)
+			(type default)
+		)
+	)
+	(wire
+		(pts
 			(xy 111.76 43.18) (xy 127 43.18)
 		)
@@
 		(pts
 			(xy 111.76 40.64) (xy 127 40.64)
+		)
+		(stroke
+			(width 0)
+			(type default)
+		)
+	)
+	(wire
+		(pts
+			(xy 111.76 35.56) (xy 127 35.56)
 		)
 		(stroke
@@
 			(effects
 				(font
+					(size 1.27 1.27)
+				)
+				(justify right)
+			)
+		)
+		(pin "I2C_INT" input
+			(at 111.76 38.1 0)
+			(effects
+				(font
+					(size 1.27 1.27)
+				)
+				(justify right)
+			)
+		)
+		(pin "I2C_RESET" output
+			(at 111.76 35.56 0)
+			(effects
+				(font
